File: design.kicad_sch (KiCad schematic)
At the start: 14 parts, among them J1 Conn_01x02, J2 Conn_01x02, J3 Conn_01x03, J4 Conn_01x03, U1 TPS61099YFFT

Commit message: init
Parts:
- removed C1, C2, C3, C4: C_Small, Capacitor_SMD:C_0805_2012Metric, symbol Device:C_Small
- removed J1, J2: Conn_01x02, Connector_PinHeader_2.54mm:PinHeader_1x02_P2.54mm_Vertical, symbol Connector_Generic:Conn_01x02
- removed J3, J4: Conn_01x03, Connector_PinHeader_2.54mm:PinHeader_1x03_P2.54mm_Vertical, symbol Connector_Generic:Conn_01x03
- removed JP1, JP2: SolderJumper_2_Open, Jumper:SolderJumper-2_P1.3mm_Open_RoundedPad1.0x1.5mm, symbol Jumper:SolderJumper_2_Open
- removed L1: L_Small, Inductor_SMD:L_1008_2520Metric, symbol Device:L_Small
- removed R1, R2: R_Small, Resistor_SMD:R_0805_2012Metric, symbol Device:R_Small
- removed U1: TPS61099YFFT, Converter_DCDC_custom:BGA6N40P3X2_122X88X62N, symbol Converter_DCDC_custom:TPS61099YFFT
- added J?: USB4130-GF-C, Connector_USB_custom:USB_C_Receptacle_GCT_USB4130-GF-C, symbol Connector_custom:USB4130-GF-C
Connections:
- new net: J?.A12 (GND), J?.B12 (GND)
- new net: J?.A9 (VBUS), J?.B9 (VBUS)
