File: design.kicad_pcb (KiCad board)
At the start: 2 copper layers, 25 x 22.9 mm, 1 part, among them J1 USB4130-GF-C

Commit message: PCB&SCH update
Parts:
- added C1: 1uF, Capacitor_SMD:C_0805_2012Metric, F.Cu at (135.0, 98.0)
- added C2: 1uF, Capacitor_SMD:C_0805_2012Metric, F.Cu at (135.0, 92.0)
- added C3: 10uF, Capacitor_SMD:C_0805_2012Metric, F.Cu at (136.0, 89.0)
- added C4: 0.1uF, Capacitor_SMD:C_0805_2012Metric, F.Cu at (138.0, 89.0)
- added C5: 1uF, Capacitor_SMD:C_0805_2012Metric, F.Cu at (167.0, 98.0)
- added C6: 100nF, Capacitor_SMD:C_0805_2012Metric, F.Cu at (146.0, 108.0)
- added C7: 0-50pF, Capacitor_SMD:C_0805_2012Metric, F.Cu at (137.0, 107.7)
- added D1: LED, LED_SMD:LED_0603_1608Metric, F.Cu at (139.0, 99.0)
- added JP1: TOG, Jumper:SolderJumper-2_P1.3mm_Open_RoundedPad1.0x1.5mm, F.Cu at (146.1, 105.0)
- added JP2: AHLB, Jumper:SolderJumper-2_P1.3mm_Open_RoundedPad1.0x1.5mm, F.Cu at (146.1, 111.0)
- added R1: 10K, Resistor_SMD:R_0805_2012Metric, F.Cu at (135.0, 105.0)
- added R2: 10K, Resistor_SMD:R_0805_2012Metric, F.Cu at (164.0, 111.0)
- added R3: 470, Resistor_SMD:R_0805_2012Metric, F.Cu at (139.0, 103.0)
- added R4: 10K, Resistor_SMD:R_0805_2012Metric, F.Cu at (159.0, 108.0)
- added R5: 10K, Resistor_SMD:R_0805_2012Metric, F.Cu at (164.0, 91.0)
- added R6: 10K, Resistor_SMD:R_0805_2012Metric, F.Cu at (162.0, 91.0)
- added R7: 5.1k, Resistor_SMD:R_0805_2012Metric, F.Cu at (143.0, 116.0)
- added R8: 5.1k, Resistor_SMD:R_0805_2012Metric, F.Cu at (157.0, 116.0)
- added SW1: EN, Button_Switch_SMD:SW_SPST_EVPBF, F.Cu at (164.0, 105.0)
- added SW2: IO9, Button_Switch_SMD:SW_SPST_EVPBF, F.Cu at (152.3, 108.0)
- added TP1: GND, TestPoint:TestPoint_Pad_D2.5mm, F.Cu at (141.0, 112.0)
- added TP2: D-, TestPoint:TestPoint_Pad_D2.5mm, F.Cu at (163.8, 98.6)
- added TP3: D+, TestPoint:TestPoint_Pad_D2.5mm, F.Cu at (163.8, 94.8)
- added TP4: +BATT, TestPoint:TestPoint_Pad_D2.5mm, F.Cu at (159.0, 112.0)
- added TP5: +3.3V, TestPoint:TestPoint_Pad_D2.5mm, F.Cu at (162.0, 87.0)
- added U1: MCP1700-3302E_SOT23, Package_TO_SOT_SMD:SOT-23, F.Cu at (135.0, 94.7)
- added U2: TCK108AF,LF, Package_TO_SOT_SMD:SOT-23-5, F.Cu at (135.2, 102.0)
- added U3: ESP32-C3-WROOM-02-N4, MCU_Espressif_custom:MODULE_ESP32-C3-WROOM-02-H4, F.Cu at (150.1, 93.1)
- added U4: TTP223, Package_TO_SOT_SMD:SOT-23-6_Handsoldering, F.Cu at (141.4, 107.2)
- moved J1 20.3 mm to (150.0, 116.0)
Connections:
- net Net-(J1-PadA12) renamed GND
- net Net-(J1-PadA9) renamed +BATT
- J1 pad A5: unconnected-(J1-PadA5) -> Net-(J1-PadA5)
- J1 pad B5: unconnected-(J1-PadB5) -> Net-(J1-PadB5)
Other:
- board size 25 x 22.9 mm -> 40 x 40 mm

Commit message: PCB design
Parts:
- moved R6 23.7 mm to (138.5, 94.0)
- moved R2 5.00 mm to (160.0, 108.0), turned to -90 degrees
- moved TP3 1.88 mm to (162.0, 94.2)
- moved TP2 1.21 mm to (162.8, 98.0)
- moved C7 1.18 mm to (137.8, 106.8)
- moved R4 1.12 mm to (157.9, 108.0)
- moved R1 0.75 mm to (134.2, 105.0)
- moved C3 0.75 mm to (136.8, 89.0)
- moved C4 0.75 mm to (138.8, 89.0)
- moved SW1 0.71 mm to (164.5, 104.5)
- moved U4 0.30 mm to (141.4, 107.5)
- moved C6 0.25 mm to (146.0, 107.8)
Routing:
- net +3.3V: track 0.00 -> 60.8 mm, vias 0 -> 2
- net +BATT: track 0.00 -> 55.6 mm
- net /EN: track 0.00 -> 48.7 mm, vias 0 -> 2
- net IO9: track 0.00 -> 29.7 mm
- net IO6: track 0.00 -> 27.6 mm
- net IO8: track 0.00 -> 9.30 mm
- net Net-(J1-PadB5): track 0.00 -> 8.92 mm
- net Net-(J1-PadA5): track 0.00 -> 8.92 mm
- net Net-(C1-Pad1): track 0.00 -> 6.41 mm
- net IO2: track 0.00 -> 5.72 mm
- net Net-(JP2-Pad1): track 0.00 -> 4.28 mm, vias 0 -> 2
- net D-: track 0.00 -> 4.06 mm
- net Net-(JP1-Pad1): track 0.00 -> 4.05 mm
- net D+: track 0.00 -> 4.00 mm
- net touch_point_1: track 0.00 -> 3.91 mm, vias 0 -> 1
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- added copper zone on F.Cu, net GND
- added copper zone on B.Cu, net touch_point_1

Commit message: PCB design
Parts:
- moved TP2 1.80 mm to (164.2, 97.0)
- moved C2 0.25 mm to (135.0, 91.8)
- moved C5 0.25 mm to (167.2, 98.0)
Routing:
- net D-: track 4.06 -> 5.73 mm

Commit message: SCH handle all ERC error warnings
Parts:
- U1: value MCP1700-3302E_SOT23 -> MCP1700x-330xxTT
Connections:
- net IO6 renamed PWR_control
- U3 pad 10: IO10 -> unconnected-(U3-Pad10)
- U3 pad 11: MCU_RX -> unconnected-(U3-Pad11)
- U3 pad 12: MCU_TX -> unconnected-(U3-Pad12)
- U3 pad 15: IO3 -> unconnected-(U3-Pad15)
- U3 pad 17: IO1 -> unconnected-(U3-Pad17)
- U3 pad 18: IO0 -> unconnected-(U3-Pad18)
- U3 pad 3: IO4 -> unconnected-(U3-Pad3)
- U3 pad 4: IO5 -> unconnected-(U3-Pad4)
Changed lines of the file:
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@@
   (net 7 "IO7")
   (net 8 "Net-(JP1-Pad1)")
-  (net 9 "IO6")
+  (net 9 "PWR_control")
   (net 10 "IO9")
   (net 11 "IO2")
@@
   (net 14 "D+")
   (net 15 "unconnected-(U2-Pad4)")
-  (net 16 "IO4")
-  (net 17 "IO5")
-  (net 18 "IO10")
-  (net 19 "MCU_RX")
-  (net 20 "MCU_TX")
-  (net 21 "IO3")
-  (net 22 "IO1")
-  (net 23 "IO0")
+  (net 16 "unconnected-(U3-Pad3)")
+  (net 17 "unconnected-(U3-Pad4)")
+  (net 18 "unconnected-(U3-Pad10)")
+  (net 19 "unconnected-(U3-Pad11)")
+  (net 20 "unconnected-(U3-Pad12)")
+  (net 21 "unconnected-(U3-Pad15)")
+  (net 22 "unconnected-(U3-Pad17)")
+  (net 23 "unconnected-(U3-Pad18)")
   (net 24 "Net-(JP2-Pad1)")
   (net 25 "Net-(C1-Pad1)")
@@
     (fp_line (start 0.9 -1.55) (end -0.25 -1.55) (layer "F.Fab") (width 0.1))
     (pad "1" smd rect (at -1.35 -0.95) (size 1.56 0.65) (layers "F.Cu" "F.Paste" "F.Mask")
-      (net 9 "IO6") (pinfunction "Q") (pintype "output"))
+      (net 9 "PWR_control") (pinfunction "Q") (pintype "output"))
     (pad "2" smd rect (at -1.35 0) (size 1.56 0.65) (layers "F.Cu" "F.Paste" "F.Mask")
       (net 2 "GND") (pinfunction "GND") (pintype "power_in"))
@@
     (fp_line (start 0.8 1.45) (end -0.8 1.45) (layer "F.Fab") (width 0.1))
     (pad "1" smd roundrect (at -1.1375 -0.95) (size 1.325 0.6) (layers "F.Cu" "F.Paste" "F.Mask") (roundrect_rratio 0.25)
-      (net 25 "Net-(C1-Pad1)") (pinfunction "VOUT") (pintype "output"))
+      (net 25 "Net-(C1-Pad1)") (pinfunction "VOUT") (pintype "power_out"))
     (pad "2" smd roundrect (at -1.1375 0) (size 1.325 0.6) (layers "F.Cu" "F.Paste" "F.Mask") (roundrect_rratio 0.25)
       (net 2 "GND") (pinfunction "GND") (pintype "input"))
     (pad "3" smd roundrect (at -1.1375 0.95) (size 1.325 0.6) (layers "F.Cu" "F.Paste" "F.Mask") (roundrect_rratio 0.25)
-      (net 9 "IO6") (pinfunction "Control") (pintype "input"))
+      (net 9 "PWR_control") (pinfunction "Control") (pintype "input"))
     (pad "4" smd roundrect (at 1.1375 0.95) (size 1.325 0.6) (layers "F.Cu" "F.Paste" "F.Mask") (roundrect_rratio 0.25)
       (net 15 "unconnected-(U2-Pad4)") (pinfunction "NC") (pintype "no_connect"))
@@
       (effects (font (size 1 1) (thickness 0.15)))
     )
-    (fp_text value "MCP1700-3302E_SOT23" (at 0 2.4) (layer "F.Fab")
+    (fp_text value "MCP1700x-330xxTT" (at 0 2.4) (layer "F.Fab")
       (effects (font (size 1 1) (thickness 0.15)))
     )
@@
       (net 4 "/EN") (pinfunction "EN") (pintype "input"))
     (pad "3" smd rect (at -8.75 0.1) (size 1.5 0.9) (layers "F.Cu" "F.Paste" "F.Mask")
-      (net 16 "IO4") (pinfunction "IO4") (pintype "bidirectional"))
+      (net 16 "unconnected-(U3-Pad3)") (pinfunction "IO4") (pintype "bidirectional+no_connect"))
     (pad "4" smd rect (at -8.75 1.6) (size 1.5 0.9) (layers "F.Cu" "F.Paste" "F.Mask")
-      (net 17 "IO5") (pinfunction "IO5") (pintype "bidirectional"))
+      (net 17 "unconnected-(U3-Pad4)") (pinfunction "IO5") (pintype "bidirectional+no_connect"))
     (pad "5" smd rect (at -8.75 3.1) (size 1.5 0.9) (layers "F.Cu" "F.Paste" "F.Mask")
-      (net 9 "IO6") (pinfunction "IO6") (pintype "bidirectional"))
+      (net 9 "PWR_control") (pinfunction "IO6") (pintype "bidirectional"))
     (pad "6" smd rect (at -8.75 4.6) (size 1.5 0.9) (layers "F.Cu" "F.Paste" "F.Mask")
       (net 7 "IO7") (pinfunction "IO7") (pintype "bidirectional"))
@@
       (net 2 "GND") (pinfunction "GND") (pintype "power_in"))
     (pad "10" smd rect (at 8.75 9.1) (size 1.5 0.9) (layers "F.Cu" "F.Paste" "F.Mask")
-      (net 18 "IO10") (pinfunction "IO10") (pintype "bidirectional"))
+      (net 18 "unconnected-(U3-Pad10)") (pinfunction "IO10") (pintype "bidirectional+no_connect"))
     (pad "11" smd rect (at 8.75 7.6) (size 1.5 0.9) (layers "F.Cu" "F.Paste" "F.Mask")
-      (net 19 "MCU_RX") (pinfunction "RXD") (pintype "bidirectional"))
+      (net 19 "unconnected-(U3-Pad11)") (pinfunction "RXD") (pintype "bidirectional+no_connect"))
     (pad "12" smd rect (at 8.75 6.1) (size 1.5 0.9) (layers "F.Cu" "F.Paste" "F.Mask")
-      (net 20 "MCU_TX") (pinfunction "TXD") (pintype "bidirectional"))
+      (net 20 "unconnected-(U3-Pad12)") (pinfunction "TXD") (pintype "bidirectional+no_connect"))
     (pad "13" smd rect (at 8.75 4.6) (size 1.5 0.9) (layers "F.Cu" "F.Paste" "F.Mask")
       (net 13 "D-") (pinfunction "IO18") (pintype "bidirectional"))
@@
       (net 14 "D+") (pinfunction "IO19") (pintype "bidirectional"))
     (pad "15" smd rect (at 8.75 1.6) (size 1.5 0.9) (layers "F.Cu" "F.Paste" "F.Mask")
-      (net 21 "IO3") (pinfunction "IO3") (pintype "bidirectional"))
+      (net 21 "unconnected-(U3-Pad15)") (pinfunction "IO3") (pintype "bidirectional+no_connect"))
     (pad "16" smd rect (at 8.75 0.1) (size 1.5 0.9) (layers "F.Cu" "F.Paste" "F.Mask")
       (net 11 "IO2") (pinfunction "IO2") (pintype "bidirectional"))
     (pad "17" smd rect (at 8.75 -1.4) (size 1.5 0.9) (layers "F.Cu" "F.Paste" "F.Mask")
-      (net 22 "IO1") (pinfunction "IO1") (pintype "bidirectional"))
+      (net 22 "unconnected-(U3-Pad17)") (pinfunction "IO1") (pintype "bidirectional+no_connect"))
     (pad "18" smd rect (at 8.75 -2.9) (size 1.5 0.9) (layers "F.Cu" "F.Paste" "F.Mask")
-      (net 23 "IO0") (pinfunction "IO0") (pintype "bidirectional"))
+      (net 23 "unconnected-(U3-Pad18)") (pinfunction "IO0") (pintype "bidirectional+no_connect"))
     (pad "19" smd rect (at -0.14 2.2) (size 0.7 0.7) (layers "F.Cu" "F.Paste" "F.Mask")
       (net 2 "GND") (pinfunction "GND") (pintype "power_in"))
@@
     (fp_line (start 1 0.625) (end -1 0.625) (layer "F.Fab") (width 0.1))
     (pad "1" smd roundrect (at -0.9125 0) (size 1.025 1.4) (layers "F.Cu" "F.Paste" "F.Mask") (roundrect_rratio 0.243902)
-      (net 9 "IO6") (pintype "passive"))
+      (net 9 "PWR_control") (pintype "passive"))
     (pad "2" smd roundrect (at 0.9125 0) (size 1.025 1.4) (layers "F.Cu" "F.Paste" "F.Mask") (roundrect_rratio 0.243902)
       (net 2 "GND") (pintype "passive"))
