File: design.kicad_pcb (KiCad board)
At the start: 2 copper layers, 40 x 40 mm, 30 parts, among them J1 USB4130-GF-C, SW1 EN, SW2 IO9, U1 MCP1700x-330xxTT, U2 TCK108AF,LF, U3 ESP32-C3-WROOM-02-N4, U4 TTP223

Commit message: changes SCH PCB
Parts:
- added C8: 1uF, Capacitor_SMD:C_0805_2012Metric, F.Cu at (218.0, 87.0)
- added C9: 1uF, Capacitor_SMD:C_0805_2012Metric, F.Cu at (218.0, 84.0)
- added D2: D_Small, Diode_SMD:D_SOD-323, F.Cu at (177.0, 102.0)
- added J2: SKEDD:490107670612, Connector_custom:WURTH_490107670612, F.Cu at (205.0, 96.5)
- added SW3: 5V/3.3V, Button_Switch_SMD:SW_DPDT_CK_JS202011JCQN, F.Cu at (188.0, 91.0)
- added SW4: VDD/NC, Button_Switch_SMD:SW_DPDT_CK_JS202011JCQN, F.Cu at (188.0, 96.5)
- added U5: MCP1700x-330xxTT, Package_TO_SOT_SMD:SOT-23, F.Cu at (213.3, 84.7)
- J1: value USB4130-GF-C -> HRO_TYPE-C-31-M-12; footprint Connector_USB_custom:USB_C_Receptacle_GCT_USB4130-GF-C -> Connector_USB:USB_C_Receptacle_HRO_TYPE-C-31-M-12
- SW1, SW2: footprint Button_Switch_SMD:SW_SPST_EVPBF -> Button_Switch_SMD_custom:RKB2
- moved J1 85.1 mm to (232.5, 95.0), turned to 90 degrees
- moved R7 82.7 mm to (222.0, 91.5), turned to -90 degrees
- moved R8 67.1 mm to (222.0, 99.5)
- moved SW2 62.4 mm to (213.5, 96.0)
- moved SW1 50.0 mm to (214.5, 103.5)
- moved TP1 31.0 mm to (172.0, 111.5)
- moved TP4 18.0 mm to (141.0, 113.0)
Connections:
- net Net-(C1-Pad1) renamed USB_input
- C5 pad 1: /EN -> MCU_EN
- J1 pad A5: Net-(J1-PadA5) -> /CC1
- J1 pad A9: +BATT -> VBUS
- J1 pad B5: Net-(J1-PadB5) -> /CC2
- J1 pad B9: +BATT -> VBUS
- J1 pad S1: unconnected-(J1-PadS1) -> GND
- R2 pad 2: /EN -> MCU_EN
- R7 pad 1: Net-(J1-PadA5) -> GND
- R7 pad 2: GND -> /CC2
- R8 pad 1: Net-(J1-PadB5) -> GND
- R8 pad 2: GND -> /CC1
- SW1 pad 1: GND -> unconnected-(SW1-Pad1)
- SW1 pad 2: /EN -> unconnected-(SW1-Pad2)
- SW2 pad 1: GND -> unconnected-(SW2-Pad1)
- SW2 pad 2: IO9 -> unconnected-(SW2-Pad2)
- U3 pad 13: D- -> MCU_D-
- U3 pad 14: D+ -> MCU_D+
- U3 pad 2: /EN -> MCU_EN
- U4 pad 1: PWR_control -> Net-(D2-Pad2)
Routing:
- net MCU_EN: track 0.00 -> 48.5 mm, vias 0 -> 2
- net /EN: track 48.5 -> 0.00 mm, vias 2 -> 0
- net +BATT: track 55.6 -> 29.1 mm
- net Net-(J1-PadB5): track 8.92 -> 0.00 mm
- net Net-(J1-PadA5): track 8.92 -> 0.00 mm
- net IO9: track 29.7 -> 22.3 mm

Commit message: more update PCB SCH
Parts:
- removed TP2: D-, TestPoint:TestPoint_Pad_D2.5mm
- removed TP3: D+, TestPoint:TestPoint_Pad_D2.5mm
- added C10: 1uF, Capacitor_SMD:C_0805_2012Metric, F.Cu at (131.4, 97.1)
- added C11: 1uF, Capacitor_SMD:C_0805_2012Metric, F.Cu at (131.4, 99.2)
- added J3: Conn_02x03_Odd_Even, Connector_PinHeader_2.54mm:PinHeader_2x03_P2.54mm_Vertical, F.Cu at (199.6, 91.0)
- moved D2 43.4 mm to (134.0, 107.5)
- moved J2 36.0 mm to (169.1, 98.9)
- moved SW3 24.2 mm to (210.8, 99.0), turned to 180 degrees
- moved SW4 24.2 mm to (210.8, 104.5)
- moved U5 22.4 mm to (222.8, 105.0)
- moved C9 21.1 mm to (219.4, 105.0), turned to 90 degrees
- moved TP1 18.6 mm to (153.5, 113.0)
- moved C8 15.7 mm to (222.8, 102.0), turned to 180 degrees
- moved C5 14.6 mm to (154.7, 105.5), turned to -90 degrees
- moved SW1 14.5 mm to (209.6, 89.8), turned to 180 degrees
- moved R2 7.81 mm to (152.6, 105.5), turned to 90 degrees
- moved R4 7.79 mm to (150.5, 105.5), turned to 90 degrees
- moved SW2 7.43 mm to (217.6, 89.8), turned to 180 degrees
- moved R8 2.12 mm to (223.5, 98.0)
- moved R7 1.50 mm to (223.5, 91.5)
Connections:
- C9 pad 1: +3.3V -> +3V3
- SW1 pad 1: unconnected-(SW1-Pad1) -> Ex_EN
- SW1 pad 2: unconnected-(SW1-Pad2) -> GND
- SW2 pad 1: unconnected-(SW2-Pad1) -> Ex_IO9
- SW2 pad 2: unconnected-(SW2-Pad2) -> GND
- SW3 pad 3: +3.3V -> +3V3
- U5 pad 2: +3.3V -> +3V3
Routing:
- net D-: track 5.73 -> 38.3 mm, vias 0 -> 2
- net VBUS: track 0.00 -> 29.7 mm
- net IO9: track 22.3 -> 48.4 mm
- net D+: track 4.00 -> 29.6 mm
- net +3.3V: track 60.7 -> 81.5 mm
- net Ex_IO9: track 0.00 -> 16.8 mm
- net +3V3: track 0.00 -> 15.9 mm
- net VDD: track 0.00 -> 14.2 mm
- net MCU_D-: track 0.00 -> 9.25 mm
- net MCU_D+: track 0.00 -> 9.21 mm
- net Ex_EN: track 0.00 -> 9.15 mm
- net MCU_EN: track 48.5 -> 41.7 mm
- net Net-(SW3-Pad2): track 0.00 -> 6.48 mm, vias 0 -> 2
- net /CC2: track 0.00 -> 5.30 mm
- net /CC1: track 0.00 -> 5.30 mm
Other:
- board size 40 x 40 mm -> 112.2 x 38.6 mm

Commit message: Update design.kicad_pcb
Parts:
- moved C8 1.28 mm to (224.0, 102.0)
- moved C9 1.28 mm to (220.7, 105.0)
- moved J1 1.28 mm to (233.8, 95.0)
- moved J3 1.28 mm to (200.9, 91.0)
- moved R7 1.28 mm to (224.8, 91.5)
- moved R8 1.28 mm to (224.8, 98.0)
- moved SW1 1.28 mm to (210.9, 89.8)
- moved SW2 1.28 mm to (218.9, 89.8)
- moved SW3 1.28 mm to (212.1, 99.0)
- moved SW4 1.28 mm to (212.1, 104.5)
- moved U5 1.28 mm to (224.1, 105.0)
Routing:
- net GND: track 0.00 -> 3.33 mm, vias 0 -> 2
- net +BATT: track 29.1 -> 31.6 mm
- net +3.3V: track 81.5 -> 80.0 mm
